Commit message: applied ouster lidar

File: APROS/urdf/iae_patrol_v1.urdf (robot description, URDF)
Before this commit: robot iae_patrol_v1, 15 links, 14 joints
Links:
- added link mission_module_link; collision box size=2.000 0.300 0.240; visual box size=0.200 0.300 0.240
- added link mission_pan_link
- added link ouster_link; visual cylinder length=0.073 radius=0.0425
Joints:
- added joint mission_pan_joint: type revolute, parent mast_stage6_link, child mission_pan_link, origin xyz=0.0 0.0 1.80 rpy=0 0 0, axis 0 0 1, limit lower=-3.14159 upper=3.14159 effort=500.0 velocity=1.0
- added joint mission_tilt_joint: type revolute, parent mission_pan_link, child mission_module_link, origin xyz=0.0 0.0 0.0 rpy=0 0 0, axis 0 1 0, limit lower=-1.5708 upper=1.5708 effort=500.0 velocity=1.0
- added joint ouster_joint: type fixed, parent mission_module_link, child ouster_link, origin xyz=0.0 0.0355 0.240 rpy=1.5708 0 0

Commit message: update

File: APROS/urdf/iae_patrol_v1.urdf (robot description, URDF)
Before this commit: robot iae_patrol_v1, 18 links, 17 joints
Joints:
- joint front_left_steer_joint: origin xyz=0.575 0.38 -0.0661 rpy=0 0 0 -> xyz=0.575 0.417 -0.0661 rpy=0 0 0
- joint front_right_steer_joint: origin xyz=0.575 -0.38 -0.0661 rpy=0 0 0 -> xyz=0.575 -0.417 -0.0661 rpy=0 0 0
- joint rear_left_wheel_joint: origin xyz=-0.575 0.38 -0.0661 rpy=-1.5708 0 0 -> xyz=-0.575 0.417 -0.0661 rpy=-1.5708 0 0

Commit message: fixed height

File: APROS/urdf/iae_patrol_v1.urdf (robot description, URDF)
Before this commit: robot iae_patrol_v1, 18 links, 17 joints
Joints:
- joint mast_base_joint: origin xyz=0.0 0.0 0.32 rpy=0 0 0 -> xyz=0.0 0.0 0.78 rpy=0 0 0
- joint mast_joint: origin xyz=0.0 0.0 0.32 rpy=0 0 0 -> xyz=0.0 0.0 0.78 rpy=0 0 0

Commit message: update

File: APROS/urdf/iae_patrol_v1.urdf (robot description, URDF)
Before this commit: robot iae_patrol_v1, 18 links, 17 joints
Joints:
- joint ouster_joint: origin xyz=0.0 0.0355 0.240 rpy=1.5708 0 0 -> xyz=0.0 0.0355 0.240 rpy=1.57079632679 0 3.14159265359

File: APROS/urdf/iae_patrol_v2.urdf (robot description, URDF)
Before this commit: robot iae_patrol_v2, 18 links, 17 joints
Links:
- added link ouster_link; visual cylinder length=0.073 radius=0.0425
Joints:
- added joint ouster_joint: type fixed, parent mission_module_link, child ouster_link, origin xyz=0.0 0.0355 0.240 rpy=1.57079632679 0 3.14159265359

Commit message: updated

File: APROS/urdf/iae_patrol_v1.urdf (robot description, URDF)
Before this commit: robot iae_patrol_v1, 18 links, 17 joints
Joints:
- joint front_left_steer_joint: limit lower=-0.4886 upper=0.4886 effort=500.0 velocity=1.0 -> lower=-0.523599 upper=0.523599 effort=500.0 velocity=0.261799
- joint front_right_steer_joint: limit lower=-0.4886 upper=0.4886 effort=500.0 velocity=1.0 -> lower=-0.523599 upper=0.523599 effort=500.0 velocity=0.261799
- joint front_steer_joint: limit lower=-0.4886 upper=0.4886 effort=500.0 velocity=1.0 -> lower=-0.523599 upper=0.523599 effort=500.0 velocity=0.261799
